Commit message: latest working with lidar except wheels

File: data/project_ws/src/ros_gz_example_description/models/diff_drive_urdf/model.urdf.xacro (robot description, xacro)
@@ -234,5 +234,5 @@
   </joint>
   <link name="lidar_link">
-    <origin rpy="0 0 0" xyz="0 0 0.25"/>
+    <origin rpy="0 0 3.14" xyz="0 0 0.25"/>
     <inertial>
       <mass value="0.1"/>
@@ -288,5 +288,5 @@
     <parent link="base_link"/>
     <child link="lidar_link"/>
-    <origin rpy="0 0 0" xyz="0 0 0.25"/>
+    <origin rpy="0 0 3.14" xyz="0 0 0.25"/>
   </joint>
 </robot>

Commit message: update

File: data/project_ws/src/ros_gz_example_description/models/diff_drive_urdf/model.urdf.xacro (robot description, xacro)
@@ -11,4 +11,7 @@
       <hardware>
         <plugin>hardware_link2/HardwareLinkInterface</plugin>
+        <param name="device">/dev/ttyUSB1</param>
+        <param name="baud_rate">115200</param>
+        <param name="timeout_ms">1000</param>
       </hardware>
     </xacro:if>
@@ -45,5 +48,5 @@
     <visual>
       <geometry>
-        <box size="0.3 0.3 0.15"/>
+        <box size="0.2 0.2 0.15"/>
       </geometry>
       <gazebo>
@@ -57,5 +60,5 @@
     <collision name='collision_chassis'>
       <geometry>
-        <box size="0.3 0.3 0.15"/>
+        <box size="0.2 0.2 0.15"/>
       </geometry>
     </collision>
@@ -67,5 +70,5 @@
   </joint>
   <link name="left_wheel">
-    <origin rpy="-1.5707 0 0" xyz="0.05 0.15 0.10"/>
+    <origin rpy="-1.5707 0 0" xyz="0.05 0.11 0.10"/>
     <inertial>
       <mass value="0.3"/>
@@ -74,5 +77,5 @@
     <visual>
       <geometry>
-        <cylinder length="0.03" radius="0.05"/>
+        <cylinder length="0.03" radius="0.034"/>
       </geometry>
       <gazebo>
@@ -86,5 +89,5 @@
     <collision name='collision_left_wheel'>
       <geometry>
-        <cylinder length="0.03" radius="0.05"/>
+        <cylinder length="0.03" radius="0.034"/>
       </geometry>
     </collision>
@@ -104,8 +107,8 @@
     <child link="left_wheel"/>
     <axis xyz="0 0 1"/>
-    <origin rpy="-1.5707 0 0" xyz="0.05 0.15 0.10"/>
+    <origin rpy="-1.5707 0 0" xyz="0.05 0.11 0.10"/>
   </joint>
   <link name="right_wheel">
-    <origin rpy="-1.5707 0 0" xyz="0.05 -0.15 0.10"/>
+    <origin rpy="-1.5707 0 0" xyz="0.05 -0.11 0.10"/>
     <inertial>
       <mass value="0.3"/>
@@ -114,5 +117,5 @@
     <visual>
       <geometry>
-        <cylinder length="0.03" radius="0.05"/>
+        <cylinder length="0.03" radius="0.034"/>
       </geometry>
       <gazebo>
@@ -126,5 +129,5 @@
     <collision name='collision_right_wheel'>
       <geometry>
-        <cylinder length="0.03" radius="0.05"/>
+        <cylinder length="0.03" radius="0.034"/>
       </geometry>
     </collision>
@@ -144,8 +147,8 @@
     <child link="right_wheel"/>
     <axis xyz="0 0 1"/>
-    <origin rpy="-1.5707 0 0" xyz="0.05 -0.15 0.10"/>
+    <origin rpy="-1.5707 0 0" xyz="0.05 -0.11 0.10"/>
   </joint>
   <link name="caster">
-    <origin rpy="0 0 0" xyz="-0.15 0 0.10"/>
+    <origin rpy="0 0 0" xyz="-0.10 0 0.10"/>
     <inertial>
       <mass value="0.005"/>
@@ -183,8 +186,8 @@
     <parent link="base_link"/>
     <child link="caster"/>
-    <origin rpy="0 0 0" xyz="-0.15 0 0.10"/>
+    <origin rpy="0 0 0" xyz="-0.10 0 0.10"/>
   </joint>
   <link name="camera_link">
-    <origin rpy="0 0 0" xyz="0.15 0 0.2"/>
+    <origin rpy="0 0 0" xyz="0.10 0 0.2"/>
     <inertial>
       <mass value="0.1"/>
@@ -231,5 +234,5 @@
     <parent link="base_link"/>
     <child link="camera_link"/>
-    <origin rpy="0 0 0" xyz="0.15 0 0.2"/>
+    <origin rpy="0 0 0" xyz="0.10 0 0.2"/>
   </joint>
   <link name="lidar_link">

Commit message: simulator update

File: data/project_ws/src/ros_gz_example_description/models/diff_drive_urdf/model.urdf.xacro (robot description, xacro)
@@ -1,5 +1,5 @@
 <?xml version="1.0"?>
 <robot name="diff_drive" xmlns:xacro="http://www.ros.org/wiki/xacro">
-  <xacro:property name="is_sim" value='False' />
+  <xacro:property name="is_sim" value='True' />
   <ros2_control name="IgnitionSystem" type="system">
     <xacro:if value="${is_sim==True}">
@@ -157,5 +157,5 @@
     <visual>
       <geometry>
-        <sphere radius="0.05"/>
+        <sphere radius="0.034"/>
       </geometry>
       <gazebo>
@@ -169,5 +169,5 @@
     <collision name='collision_caster'>
       <geometry>
-        <sphere radius="0.05"/>
+        <sphere radius="0.034"/>
       </geometry>
     </collision>

Commit message: update

File: data/project_ws/src/ros_gz_example_description/models/diff_drive_urdf/model.urdf.xacro (robot description, xacro)
@@ -1,5 +1,5 @@
 <?xml version="1.0"?>
 <robot name="diff_drive" xmlns:xacro="http://www.ros.org/wiki/xacro">
-  <xacro:property name="is_sim" value='True' />
+  <xacro:property name="is_sim" value='False' />
   <ros2_control name="IgnitionSystem" type="system">
     <xacro:if value="${is_sim==True}">

Commit message: add sim option

File: data/project_ws/src/ros_gz_example_description/models/diff_drive_urdf/model.urdf.xacro (robot description, xacro)
@@ -1,5 +1,5 @@
 <?xml version="1.0"?>
 <robot name="diff_drive" xmlns:xacro="http://www.ros.org/wiki/xacro">
-  <xacro:property name="is_sim" value='False' />
+  <xacro:property name="is_sim" value="$(arg sim_mode)" />
   <ros2_control name="IgnitionSystem" type="system">
     <xacro:if value="${is_sim==True}">

Commit message: update

File: data/project_ws/src/ros_gz_example_description/models/diff_drive_urdf/model.urdf.xacro (robot description, xacro)
@@ -37,4 +37,8 @@
       <parameters>/root/data/project_ws/src/ros_gz_example_bringup/config/diff_drive_controller_velocity.yaml</parameters>
     </plugin>
+    <plugin
+      filename="ignition-gazebo-imu-system"
+      name="gz::sim::systems::Imu">
+    </plugin>
   </gazebo>
   <link name="base_link">
@@ -293,3 +297,42 @@
     <origin rpy="0 0 3.14" xyz="0 0 0.25"/>
   </joint>
+  <link name="imu_link">
+    <origin rpy="0 0 0.15" xyz="0 0 0"/>
+    <inertial>
+      <mass value="0.1"/>
+      <inertia ixx="0.000166667" iyy="0.000166667" izz="0.000166667" ixy="0" ixz="0" iyz="0"/>
+    </inertial>
+    <visual>
+      <geometry>
+        <box size="0.05 0.05 0.05"/>
+      </geometry>
+      <gazebo>
+        <material>
+          <ambient>0 0 0 1</ambient>
+          <diffuse>0 0 0 1</diffuse>
+          <specular>0 0 0 1</specular>
+        </material>
+      </gazebo>
+    </visual>
+    <collision name="collision">
+      <geometry>
+        <box size="0.05 0.05 0.05"/>
+      </geometry>
+    </collision>
+  </link>
+  <gazebo reference="imu_link">
+    <sensor name="imu" type="imu">
+      <always_on>1</always_on>
+      <update_rate>100</update_rate>
+      <visualize>true</visualize>
+      <topic>imu</topic>
+      <enable_metrics>true</enable_metrics>
+      <ignition_frame_id>diff_drive/imu_link</ignition_frame_id>
+    </sensor>
+  </gazebo>
+  <joint name="imu_joint" type="fixed">
+    <parent link="base_link"/>
+    <child link="imu_link"/>
+    <origin rpy="0 0 0.15" xyz="0 0 0"/>
+  </joint>
 </robot>

Commit message: update

File: data/project_ws/src/ros_gz_example_description/models/diff_drive_urdf/model.urdf.xacro (robot description, xacro)
@@ -298,24 +298,16 @@
   </joint>
   <link name="imu_link">
-    <origin rpy="0 0 0.15" xyz="0 0 0"/>
-    <inertial>
-      <mass value="0.1"/>
-      <inertia ixx="0.000166667" iyy="0.000166667" izz="0.000166667" ixy="0" ixz="0" iyz="0"/>
-    </inertial>
-    <visual>
-      <geometry>
-        <box size="0.05 0.05 0.05"/>
-      </geometry>
-      <gazebo>
-        <material>
-          <ambient>0 0 0 1</ambient>
-          <diffuse>0 0 0 1</diffuse>
-          <specular>0 0 0 1</specular>
-        </material>
-      </gazebo>
+    <origin rpy="0 0 0" xyz="0 0 0.15"/>
+    <inertial>
+      <mass value="0.001"/>
+      <inertia ixx="1.67e-10" iyy="1.67e-10" izz="1.67e-10" ixy="0" ixz="0" iyz="0"/>    </inertial>
+    <visual>
+      <geometry>
+        <box size="0.001 0.001 0.001"/>
+      </geometry>
     </visual>
     <collision name="collision">
       <geometry>
-        <box size="0.05 0.05 0.05"/>
+        <box size="0.001 0.001 0.001"/>
       </geometry>
     </collision>
@@ -334,5 +326,5 @@
     <parent link="base_link"/>
     <child link="imu_link"/>
-    <origin rpy="0 0 0.15" xyz="0 0 0"/>
+    <origin rpy="0 0 0" xyz="0 0 0.15"/>
   </joint>
 </robot>

Commit message: rotate IMU 180deg

File: data/project_ws/src/ros_gz_example_description/models/diff_drive_urdf/model.urdf.xacro (robot description, xacro)
@@ -298,5 +298,5 @@
   </joint>
   <link name="imu_link">
-    <origin rpy="0 0 0" xyz="0 0 0.15"/>
+    <origin rpy="0 0 3.14" xyz="0 0 0.15"/>
     <inertial>
       <mass value="0.001"/>
@@ -326,5 +326,5 @@
     <parent link="base_link"/>
     <child link="imu_link"/>
-    <origin rpy="0 0 0" xyz="0 0 0.15"/>
+    <origin rpy="0 0 3.14" xyz="0 0 0.15"/>
   </joint>
 </robot>

Commit message: update

File: data/project_ws/src/ros_gz_example_description/models/diff_drive_urdf/model.urdf.xacro (robot description, xacro)
@@ -44,6 +44,6 @@
   <link name="base_link">
   </link>
-  <link name="chassis">
-    <origin rpy="0 0 0" xyz="0 0 0.15"/>
+  <link name="chassis_link">
+    <origin rpy="0 0 0" xyz="0 0 0.10"/>
     <inertial>
       <mass value="1"/>
@@ -70,9 +70,9 @@
   <joint name="base_joint" type="fixed">
     <parent link="base_link"/>
-    <child link="chassis"/>
-    <origin rpy="0 0 0" xyz="0 0 0.15"/>
+    <child link="chassis_link"/>
+    <origin rpy="0 0 0" xyz="0 0 0.10"/>
   </joint>
   <link name="left_wheel">
-    <origin rpy="-1.5707 0 0" xyz="0.05 0.11 0.10"/>
+    <origin rpy="-1.5707 0 0" xyz="0.05 0.11 0.05"/>
     <inertial>
       <mass value="0.3"/>
@@ -111,8 +111,8 @@
     <child link="left_wheel"/>
     <axis xyz="0 0 1"/>
-    <origin rpy="-1.5707 0 0" xyz="0.05 0.11 0.10"/>
+    <origin rpy="-1.5707 0 0" xyz="0.05 0.11 0.05"/>
   </joint>
   <link name="right_wheel">
-    <origin rpy="-1.5707 0 0" xyz="0.05 -0.11 0.10"/>
+    <origin rpy="-1.5707 0 0" xyz="0.05 -0.11 0.05"/>
     <inertial>
       <mass value="0.3"/>
@@ -151,8 +151,8 @@
     <child link="right_wheel"/>
     <axis xyz="0 0 1"/>
-    <origin rpy="-1.5707 0 0" xyz="0.05 -0.11 0.10"/>
+    <origin rpy="-1.5707 0 0" xyz="0.05 -0.11 0.05"/>
   </joint>
   <link name="caster">
-    <origin rpy="0 0 0" xyz="-0.10 0 0.10"/>
+    <origin rpy="0 0 0" xyz="-0.10 0 0.05"/>
     <inertial>
       <mass value="0.005"/>
@@ -190,8 +190,8 @@
     <parent link="base_link"/>
     <child link="caster"/>
-    <origin rpy="0 0 0" xyz="-0.10 0 0.10"/>
+    <origin rpy="0 0 0" xyz="-0.10 0 0.05"/>
   </joint>
   <link name="camera_link">
-    <origin rpy="0 0 0" xyz="0.10 0 0.2"/>
+    <origin rpy="0 0 0" xyz="0.10 0 0.15"/>
     <inertial>
       <mass value="0.1"/>
@@ -238,8 +238,8 @@
     <parent link="base_link"/>
     <child link="camera_link"/>
-    <origin rpy="0 0 0" xyz="0.10 0 0.2"/>
+    <origin rpy="0 0 0" xyz="0.10 0 0.15"/>
   </joint>
   <link name="lidar_link">
-    <origin rpy="0 0 3.14" xyz="0 0 0.25"/>
+    <origin rpy="0 0 3.14" xyz="0 0 0.20"/>
     <inertial>
       <mass value="0.1"/>
@@ -295,8 +295,8 @@
     <parent link="base_link"/>
     <child link="lidar_link"/>
-    <origin rpy="0 0 3.14" xyz="0 0 0.25"/>
+    <origin rpy="0 0 3.14" xyz="0 0 0.20"/>
   </joint>
   <link name="imu_link">
-    <origin rpy="0 0 3.14" xyz="0 0 0.15"/>
+    <origin rpy="0 0 3.14" xyz="0 0 0.10"/>
     <inertial>
       <mass value="0.001"/>
@@ -326,5 +326,5 @@
     <parent link="base_link"/>
     <child link="imu_link"/>
-    <origin rpy="0 0 3.14" xyz="0 0 0.15"/>
+    <origin rpy="0 0 3.14" xyz="0 0 0.10"/>
   </joint>
 </robot>

Commit message: update

File: data/project_ws/src/ros_gz_example_description/models/diff_drive_urdf/model.urdf.xacro (robot description, xacro)
@@ -105,5 +105,5 @@
     <collision name='collision_left_wheel'>
       <geometry>
-        <cylinder length="0.03" radius="0.034"/>
+        <cylinder length="0.02677" radius="0.033685"/>
       </geometry>
     </collision>
@@ -112,6 +112,8 @@
         <friction>
           <ode>
-            <mu>1.0</mu>
-            <mu2>1.0</mu2>
+            <mu>0.8</mu>
+            <mu2>0.9</mu2>
+            <slip1>0.3</slip1>  <!-- Longitudinal slip -->
+            <slip2>0.1</slip2>  <!-- Lateral slip -->
           </ode>
         </friction>
@@ -145,5 +147,5 @@
     <collision name='collision_right_wheel'>
       <geometry>
-        <cylinder length="0.03" radius="0.034"/>
+        <cylinder length="0.02677" radius="0.033685"/>
       </geometry>
     </collision>
@@ -152,6 +154,8 @@
         <friction>
           <ode>
-            <mu>1.0</mu>
-            <mu2>1.0</mu2>
+            <mu>0.8</mu>
+            <mu2>0.9</mu2>
+            <slip1>0.35</slip1>  <!-- Longitudinal slip -->
+            <slip2>0.1</slip2>  <!-- Lateral slip -->
           </ode>
         </friction>
@@ -333,18 +337,64 @@
       <enable_metrics>true</enable_metrics>
       <ignition_frame_id>imu_link</ignition_frame_id>
-      <!-- High Noise Parameters for "Very Bad" Sensor Simulation -->
-      <gaussianNoise>2.0</gaussianNoise> <!-- High noise level -->
-      <bias>
+      <imu>
         <angular_velocity>
-          <x>0.1</x> <!-- Large bias -->
-          <y>0.1</y> <!-- Large bias -->
-          <z>0.1</z> <!-- Large bias -->
+          <x>
+            <bias>
+              <mean>0.01</mean> <!-- Constant bias for the x-axis -->
+            </bias>
+            <noise type="gaussian">
+              <mean>0.0</mean>
+              <stddev>0.05</stddev> <!-- Increased noise for the x-axis -->
+            </noise>
+          </x>
+          <y>
+            <bias>
+              <mean>0.02</mean> <!-- Constant bias for the y-axis -->
+            </bias>
+            <noise type="gaussian">
+              <mean>0.0</mean>
+              <stddev>0.05</stddev> <!-- Increased noise for the y-axis -->
+            </noise>
+          </y>
+          <z>
+            <bias>
+              <mean>0.015</mean> <!-- Constant bias for the z-axis -->
+            </bias>
+            <noise type="gaussian">
+              <mean>0.0</mean>
+              <stddev>0.05</stddev> <!-- Increased noise for the z-axis -->
+            </noise>
+          </z>
         </angular_velocity>
         <linear_acceleration>
-          <x>0.5</x> <!-- Large bias -->
-          <y>0.5</y> <!-- Large bias -->
-          <z>0.5</z> <!-- Large bias -->
+          <x>
+            <bias>
+              <mean>0.05</mean> <!-- Constant bias for the x-axis -->
+            </bias>
+            <noise type="gaussian">
+              <mean>0.0</mean>
+              <stddev>0.3</stddev> <!-- Increased noise for the x-axis -->
+            </noise>
+          </x>
+          <y>
+            <bias>
+              <mean>0.03</mean> <!-- Constant bias for the y-axis -->
+            </bias>
+            <noise type="gaussian">
+              <mean>0.0</mean>
+              <stddev>0.3</stddev> <!-- Increased noise for the y-axis -->
+            </noise>
+          </y>
+          <z>
+            <bias>
+              <mean>0.04</mean> <!-- Constant bias for the z-axis -->
+            </bias>
+            <noise type="gaussian">
+              <mean>0.0</mean>
+              <stddev>0.3</stddev> <!-- Increased noise for the z-axis -->
+            </noise>
+          </z>
         </linear_acceleration>
-      </bias>
+      </imu>
     </sensor>
   </gazebo>

Commit message: update

File: data/project_ws/src/ros_gz_example_description/models/diff_drive_urdf/model.urdf.xacro (robot description, xacro)
@@ -53,9 +53,13 @@
       name="gz::sim::systems::Imu">
     </plugin>
+    <plugin
+      filename="ignition-gazebo-magnetometer-system"
+      name="gz::sim::systems::Magnetometer">
+    </plugin>
   </gazebo>
   <link name="base_link">
   </link>
   <link name="chassis_link">
-    <origin rpy="0 0 0" xyz="0 0 0.10"/>
+    <origin rpy="0 0 0" xyz="0 0 0"/>
     <inertial>
       <mass value="1"/>
@@ -83,8 +87,8 @@
     <parent link="base_link"/>
     <child link="chassis_link"/>
-    <origin rpy="0 0 0" xyz="0 0 0.10"/>
+    <origin rpy="0 0 0" xyz="0 0 0"/>
   </joint>
   <link name="left_wheel">
-    <origin rpy="-1.5707 0 0" xyz="0.05 0.11 0.05"/>
+    <origin rpy="-1.5707 0 0" xyz="0.05 0.11 -0.05"/>
     <inertial>
       <mass value="0.3"/>
@@ -125,8 +129,8 @@
     <child link="left_wheel"/>
     <axis xyz="0 0 1"/>
-    <origin rpy="-1.5707 0 0" xyz="0.05 0.11 0.05"/>
+    <origin rpy="-1.5707 0 0" xyz="0.05 0.11 -0.05"/>
   </joint>
   <link name="right_wheel">
-    <origin rpy="-1.5707 0 0" xyz="0.05 -0.11 0.05"/>
+    <origin rpy="-1.5707 0 0" xyz="0.05 -0.11 -0.05"/>
     <inertial>
       <mass value="0.3"/>
@@ -167,8 +171,8 @@
     <child link="right_wheel"/>
     <axis xyz="0 0 1"/>
-    <origin rpy="-1.5707 0 0" xyz="0.05 -0.11 0.05"/>
+    <origin rpy="-1.5707 0 0" xyz="0.05 -0.11 -0.05"/>
   </joint>
   <link name="caster">
-    <origin rpy="0 0 0" xyz="-0.10 0 0.05"/>
+    <origin rpy="0 0 0" xyz="-0.10 0 -0.05"/>
     <inertial>
       <mass value="0.005"/>
@@ -206,8 +210,8 @@
     <parent link="base_link"/>
     <child link="caster"/>
-    <origin rpy="0 0 0" xyz="-0.10 0 0.05"/>
+    <origin rpy="0 0 0" xyz="-0.10 0 -0.05"/>
   </joint>
   <link name="camera_link">
-    <origin rpy="0 0 0" xyz="0.10 0 0.15"/>
+    <origin rpy="0 0 0" xyz="0.10 0 0.05"/>
     <inertial>
       <mass value="0.1"/>
@@ -254,8 +258,8 @@
     <parent link="base_link"/>
     <child link="camera_link"/>
-    <origin rpy="0 0 0" xyz="0.10 0 0.15"/>
+    <origin rpy="0 0 0" xyz="0.10 0 0.05"/>
   </joint>
   <link name="lidar_link">
-    <origin rpy="0 0 3.14" xyz="0 0 0.20"/>
+    <origin rpy="0 0 3.14" xyz="0 0 0.1"/>
     <inertial>
       <mass value="0.1"/>
@@ -311,8 +315,8 @@
     <parent link="base_link"/>
     <child link="lidar_link"/>
-    <origin rpy="0 0 3.14" xyz="0 0 0.20"/>
+    <origin rpy="0 0 3.14" xyz="0 0 0.1"/>
   </joint>
   <link name="imu_link">
-    <origin rpy="0 0 3.14" xyz="0 0 0.10"/>
+    <origin rpy="0 0 3.14" xyz="0 0 0"/>
     <inertial>
       <mass value="0.001"/>
@@ -337,31 +341,31 @@
       <enable_metrics>true</enable_metrics>
       <ignition_frame_id>imu_link</ignition_frame_id>
-      <imu>
+      <!-- <imu>
         <angular_velocity>
           <x>
             <bias>
-              <mean>0.01</mean> <!-- Constant bias for the x-axis -->
-            </bias>
-            <noise type="gaussian">
-              <mean>0.0</mean>
-              <stddev>0.05</stddev> <!-- Increased noise for the x-axis -->
+              <mean>0.01</mean>
+            </bias>
+            <noise type="gaussian">
+              <mean>0.0</mean>
+              <stddev>0.05</stddev>
             </noise>
           </x>
           <y>
             <bias>
-              <mean>0.02</mean> <!-- Constant bias for the y-axis -->
-            </bias>
-            <noise type="gaussian">
-              <mean>0.0</mean>
-              <stddev>0.05</stddev> <!-- Increased noise for the y-axis -->
+              <mean>0.02</mean>
+            </bias>
+            <noise type="gaussian">
+              <mean>0.0</mean>
+              <stddev>0.05</stddev>
             </noise>
           </y>
           <z>
             <bias>
-              <mean>0.015</mean> <!-- Constant bias for the z-axis -->
-            </bias>
-            <noise type="gaussian">
-              <mean>0.0</mean>
-              <stddev>0.05</stddev> <!-- Increased noise for the z-axis -->
+              <mean>0.015</mean>
+            </bias>
+            <noise type="gaussian">
+              <mean>0.0</mean>
+              <stddev>0.05</stddev>
             </noise>
           </z>
@@ -370,31 +374,31 @@
           <x>
             <bias>
-              <mean>0.05</mean> <!-- Constant bias for the x-axis -->
-            </bias>
-            <noise type="gaussian">
-              <mean>0.0</mean>
-              <stddev>0.3</stddev> <!-- Increased noise for the x-axis -->
+              <mean>0.05</mean>
+            </bias>
+            <noise type="gaussian">
+              <mean>0.0</mean>
+              <stddev>0.3</stddev>
             </noise>
           </x>
           <y>
             <bias>
-              <mean>0.03</mean> <!-- Constant bias for the y-axis -->
-            </bias>
-            <noise type="gaussian">
-              <mean>0.0</mean>
-              <stddev>0.3</stddev> <!-- Increased noise for the y-axis -->
+              <mean>0.03</mean>
+            </bias>
+            <noise type="gaussian">
+              <mean>0.0</mean>
+              <stddev>0.3</stddev>
             </noise>
           </y>
           <z>
             <bias>
-              <mean>0.04</mean> <!-- Constant bias for the z-axis -->
-            </bias>
-            <noise type="gaussian">
-              <mean>0.0</mean>
-              <stddev>0.3</stddev> <!-- Increased noise for the z-axis -->
+              <mean>0.04</mean>
+            </bias>
+            <noise type="gaussian">
+              <mean>0.0</mean>
+              <stddev>0.3</stddev>
             </noise>
           </z>
         </linear_acceleration>
-      </imu>
+      </imu> -->
     </sensor>
   </gazebo>
@@ -402,5 +406,56 @@
     <parent link="base_link"/>
     <child link="imu_link"/>
-    <origin rpy="0 0 3.14" xyz="0 0 0.10"/>
+    <origin rpy="0 0 3.14" xyz="0 0 0"/>
+  </joint>
+  <link name="magnetometer_link">
+    <origin rpy="0 0 3.14" xyz="0 0 0"/>
+    <inertial>
+      <mass value="0.001"/>
+      <inertia ixx="1.67e-10" iyy="1.67e-10" izz="1.67e-10" ixy="0" ixz="0" iyz="0"/>    </inertial>
+    <visual>
+      <geometry>
+        <box size="0.001 0.001 0.001"/>
+      </geometry>
+    </visual>
+    <collision name="collision">
+      <geometry>
+        <box size="0.001 0.001 0.001"/>
+      </geometry>
+    </collision>
+  </link>
+  <gazebo reference="magnetometer_link">
+    <sensor name="magnetometer" type="magnetometer">
+      <always_on>1</always_on>
+      <update_rate>100</update_rate>
+      <visualize>true</visualize>
+      <topic>magnetometer</topic>
+      <ignition_frame_id>magnetometer_link</ignition_frame_id>
+      <enable_metrics>true</enable_metrics>
+      <!-- <magnetometer>
+        <x>
+          <noise type="gaussian">
+            <mean>0.0</mean>
+            <stddev>0.1</stddev>
+          </noise>
+        </x>
+        <y>
+          <noise type="gaussian">
+            <mean>0.0</mean>
+            <stddev>0.1</stddev>
+          </noise>
+        </y>
+        <z>
+          <noise type="gaussian">
+            <mean>0.0</mean>
+            <stddev>0.1</stddev>
+          </noise>
+        </z>
+      </magnetometer> -->
+    </sensor>
+  </gazebo>
+  <joint name="magnetometer_joint" type="fixed">
+    <parent link="base_link"/>
+    <child link="magnetometer_link"/>
+    <origin rpy="0 0 3.14" xyz="0 0 0"/>
   </joint>
 </robot>
