Commit message: removed imu from ros2

File: data/project_ws/src/ros_gz_example_description/models/diff_drive_urdf/model.urdf.xacro (robot description, xacro)
@@ -32,5 +32,5 @@
       <state_interface name="velocity"/>
     </joint>
-    <sensor name="imu_sensor">
+    <!-- <sensor name="imu_sensor">
       <state_interface name="orientation.x"/>
       <state_interface name="orientation.y"/>
@@ -43,5 +43,5 @@
       <state_interface name="linear_acceleration.y"/>
       <state_interface name="linear_acceleration.z"/>
-    </sensor>
+    </sensor> -->
   </ros2_control>
   <gazebo>
@@ -318,5 +318,5 @@
   </joint>
   <link name="imu_link">
-    <origin rpy="0 0 3.14" xyz="0 0 0"/>
+    <origin rpy="0 0 0" xyz="0 0 0"/>
     <inertial>
       <mass value="0.001"/>
@@ -406,8 +406,8 @@
     <parent link="base_link"/>
     <child link="imu_link"/>
-    <origin rpy="0 0 3.14" xyz="0 0 0"/>
+    <origin rpy="0 0 0" xyz="0 0 0"/>
   </joint>
   <link name="magnetometer_link">
-    <origin rpy="0 0 3.14" xyz="0 0 0"/>
+    <origin rpy="0 0 0" xyz="0 0 0"/>
     <inertial>
       <mass value="0.001"/>
@@ -457,5 +457,5 @@
     <parent link="base_link"/>
     <child link="magnetometer_link"/>
-    <origin rpy="0 0 3.14" xyz="0 0 0"/>
+    <origin rpy="0 0 0" xyz="0 0 0"/>
   </joint>
 </robot>

Commit message: update

File: data/project_ws/src/ros_gz_example_description/models/diff_drive_urdf/model.urdf.xacro (robot description, xacro)
@@ -5,5 +5,5 @@
     <xacro:if value="${is_sim==True}">
       <hardware>
-        <plugin>ign_ros2_control/IgnitionSystem</plugin>
+        <plugin>gz_ros2_control/GazeboSimSystem</plugin>
       </hardware>
     </xacro:if>
@@ -34,13 +34,13 @@
   </ros2_control>
   <gazebo>
-    <plugin filename="ign_ros2_control-system" name="ign_ros2_control::IgnitionROS2ControlPlugin">
+    <plugin filename="gz_ros2_control-system" name="gz_ros2_control::GazeboSimROS2ControlPlugin">
       <parameters>/root/data/project_ws/src/ros_gz_example_bringup/config/diff_drive_controller_velocity.yaml</parameters>
     </plugin>
     <plugin
-      filename="ignition-gazebo-imu-system"
+      filename="gz-sim-imu-system"
       name="gz::sim::systems::Imu">
     </plugin>
     <plugin
-      filename="ignition-gazebo-magnetometer-system"
+      filename="gz-sim-magnetometer-system"
       name="gz::sim::systems::Magnetometer">
     </plugin>
@@ -118,4 +118,5 @@
     <axis xyz="0 0 1"/>
     <origin rpy="-1.5707 0 0" xyz="0.05 0.11 -0.05"/>
+    <dynamics damping="0.2"/>
   </joint>
   <link name="right_wheel">
@@ -160,4 +161,5 @@
     <axis xyz="0 0 1"/>
     <origin rpy="-1.5707 0 0" xyz="0.05 -0.11 -0.05"/>
+    <dynamics damping="0.2"/>
   </joint>
   <link name="caster">
@@ -269,5 +271,5 @@
           <pose>0 0 0 0 0 0</pose>
           <topic>scan</topic>
-          <ignition_frame_id>lidar_link</ignition_frame_id>
+          <gz_frame_id>lidar_link</gz_frame_id>
           <update_rate>10</update_rate>
           <lidar>
@@ -328,65 +330,5 @@
       <topic>imu</topic>
       <enable_metrics>true</enable_metrics>
-      <ignition_frame_id>imu_link</ignition_frame_id>
-      <imu>
-        <angular_velocity>
-          <x>
-            <bias>
-              <mean>0.01</mean>
-            </bias>
-            <noise type="gaussian">
-              <mean>0.0</mean>
-              <stddev>0.05</stddev>
-            </noise>
-          </x>
-          <y>
-            <bias>
-              <mean>0.02</mean>
-            </bias>
-            <noise type="gaussian">
-              <mean>0.0</mean>
-              <stddev>0.05</stddev>
-            </noise>
-          </y>
-          <z>
-            <bias>
-              <mean>0.015</mean>
-            </bias>
-            <noise type="gaussian">
-              <mean>0.0</mean>
-              <stddev>0.05</stddev>
-            </noise>
-          </z>
-        </angular_velocity>
-        <linear_acceleration>
-          <x>
-            <bias>
-              <mean>0.05</mean>
-            </bias>
-            <noise type="gaussian">
-              <mean>0.0</mean>
-              <stddev>0.3</stddev>
-            </noise>
-          </x>
-          <y>
-            <bias>
-              <mean>0.03</mean>
-            </bias>
-            <noise type="gaussian">
-              <mean>0.0</mean>
-              <stddev>0.3</stddev>
-            </noise>
-          </y>
-          <z>
-            <bias>
-              <mean>0.04</mean>
-            </bias>
-            <noise type="gaussian">
-              <mean>0.0</mean>
-              <stddev>0.3</stddev>
-            </noise>
-          </z>
-        </linear_acceleration>
-      </imu>
+      <gz_frame_id>imu_link</gz_frame_id>
     </sensor>
   </gazebo>
@@ -418,5 +360,5 @@
       <visualize>true</visualize>
       <topic>magnetometer</topic>
-      <ignition_frame_id>magnetometer_link</ignition_frame_id>
+      <gz_frame_id>magnetometer_link</gz_frame_id>
       <enable_metrics>true</enable_metrics>
       <!-- <magnetometer>

Commit message: chnage to stereo camera

File: data/project_ws/src/ros_gz_example_description/models/diff_drive_urdf/model.urdf.xacro (robot description, xacro)
@@ -202,6 +202,6 @@
     <origin rpy="0 0 0" xyz="-0.10 0 -0.05"/>
   </joint>
-  <link name="camera_link">
-    <origin rpy="0 0 0" xyz="0.10 0 0.05"/>
+  <link name="camera_left_link">
+    <origin rpy="0 0 0" xyz="0.10 0.03 0.05"/>
     <inertial>
       <mass value="0.1"/>
@@ -210,5 +210,5 @@
     <visual>
       <geometry>
-        <box size="0.05 0.05 0.05"/>
+        <box size="0.02 0.02 0.02"/>
       </geometry>
       <gazebo>
@@ -222,29 +222,10 @@
     <collision name="collision">
       <geometry>
-        <box size="0.05 0.05 0.05"/>
-      </geometry>
-    </collision>
-  </link>
-  <!-- <gazebo reference="camera_link">
-        <sensor name="camera" type="camera">
-          <camera>
-            <horizontal_fov>2</horizontal_fov>
-            <image>
-              <width>1280</width>
-              <height>720</height>
-            </image>
-            <clip>
-              <near>0.1</near>
-              <far>100</far>
-            </clip>
-          </camera>
-          <always_on>1</always_on>
-          <update_rate>60</update_rate>
-          <visualize>1</visualize>
-          <topic>camera</topic>
-        </sensor>
-  </gazebo> -->
-  <gazebo reference="camera_link">
-        <sensor name="wide_angle_camera" type="wideanglecamera">
+        <box size="0.02 0.02 0.02"/>
+      </geometry>
+    </collision>
+  </link>
+  <gazebo reference="camera_left_link">
+        <sensor name="wide_angle_camera_left" type="wideanglecamera">
           <camera>
             <horizontal_fov>3.14</horizontal_fov>
@@ -273,11 +254,71 @@
           <update_rate>10</update_rate>
           <visualize>1</visualize>
-          <topic>camera</topic>
+          <topic>camera_left</topic>
         </sensor>
   </gazebo>
-  <joint name="camera_joint" type="fixed">
-    <parent link="base_link"/>
-    <child link="camera_link"/>
-    <origin rpy="0 0 0" xyz="0.10 0 0.05"/>
+  <joint name="camera_left_joint" type="fixed">
+    <parent link="base_link"/>
+    <child link="camera_left_link"/>
+    <origin rpy="0 0 0" xyz="0.10 0.03 0.05"/>
+  </joint>
+  <link name="camera_right_link">
+    <origin rpy="0 0 0" xyz="0.10 -0.03 0.05"/>
+    <inertial>
+      <mass value="0.1"/>
+      <inertia ixx="0.000166667" iyy="0.000166667" izz="0.000166667" ixy="0" ixz="0" iyz="0"/>
+    </inertial>
+    <visual>
+      <geometry>
+        <box size="0.02 0.02 0.02"/>
+      </geometry>
+      <gazebo>
+        <material>
+          <ambient>0 0 0 1</ambient>
+          <diffuse>0 0 0 1</diffuse>
+          <specular>0 0 0 1</specular>
+        </material>
+      </gazebo>
+    </visual>
+    <collision name="collision">
+      <geometry>
+        <box size="0.02 0.02 0.02"/>
+      </geometry>
+    </collision>
+  </link>
+  <gazebo reference="camera_right_link">
+        <sensor name="wide_angle_camera_right" type="wideanglecamera">
+          <camera>
+            <horizontal_fov>3.14</horizontal_fov>
+            <image>
+              <width>1280</width>
+              <height>720</height>
+            </image>
+            <clip>
+              <near>0.1</near>
+              <far>100</far>
+            </clip>
+            <lens>
+              <type>custom</type>
+              <custom_function>
+                <c1>1.05</c1>
+                <c2>4</c2>
+                <f>1.0</f>
+                <fun>tan</fun>
+              </custom_function>
+              <scale_to_hfov>true</scale_to_hfov>
+              <cutoff_angle>3.1415</cutoff_angle>
+              <env_texture_size>1024</env_texture_size>
+            </lens>
+          </camera>
+          <always_on>1</always_on>
+          <update_rate>10</update_rate>
+          <visualize>1</visualize>
+          <topic>camera_right</topic>
+        </sensor>
+  </gazebo>
+  <joint name="camera_right_joint" type="fixed">
+    <parent link="base_link"/>
+    <child link="camera_right_link"/>
+    <origin rpy="0 0 0" xyz="0.10 -0.03 0.05"/>
   </joint>
   <link name="lidar_link">
