Commit message: latest local camera working localization.

File: data/project_ws/src/ros_gz_example_description/models/diff_drive_urdf/model.urdf copy.xacro (robot description, xacro)
@@ -205,5 +205,5 @@
     <parent link="base_link"/>
     <child link="t265_link"/>
-    <origin rpy="1.57 0.0 -1.57" xyz="0.0 0.0 0.2"/>
+    <origin rpy="1.57 0.0 -1.57" xyz="0.0 0.0 0.5"/>
   </joint>
   <link name="t265_link">
@@ -255,11 +255,42 @@
     </collision>
   </link>
+  <gazebo reference="camera_left_link">
+        <sensor name="wide_angle_camera_left" type="wideanglecamera">
+          <camera>
+            <horizontal_fov>3.14</horizontal_fov>
+            <image>
+              <width>1280</width>
+              <height>720</height>
+            </image>
+            <clip>
+              <near>0.1</near>
+              <far>100</far>
+            </clip>
+            <lens>
+              <type>custom</type>
+              <custom_function>
+                <c1>1.05</c1>
+                <c2>4</c2>
+                <f>1.0</f>
+                <fun>tan</fun>
+              </custom_function>
+              <scale_to_hfov>true</scale_to_hfov>
+              <cutoff_angle>3.1415</cutoff_angle>
+              <env_texture_size>1024</env_texture_size>
+            </lens>
+          </camera>
+          <always_on>1</always_on>
+          <update_rate>10</update_rate>
+          <visualize>1</visualize>
+          <topic>camera_left</topic>
+        </sensor>
+  </gazebo>
   <joint name="camera_left_joint" type="fixed">
     <parent link="t265_link"/>
     <child link="camera_left_link"/>
-    <origin rpy="0 1.57 1.57" xyz="-0.0354 0 0"/>
-  </joint>
-  <link name="camera_left_optical_link">
-    <!-- <origin rpy="0 0 0" xyz="0.10 0.03 0.05"/> -->
+    <origin rpy="-3.14 0 0" xyz="-0.03 0 0"/>
+  </joint>
+  <link name="camera_right_link">
+    <!-- <origin rpy="0 0 0" xyz="0.10 -0.03 0.05"/> -->
     <inertial>
       <mass value="0.1"/>
@@ -284,113 +315,40 @@
     </collision>
   </link>
-  <joint name="camera_left_optical_joint" type="fixed">
+  <gazebo reference="camera_right_link">
+        <sensor name="wide_angle_camera_right" type="wideanglecamera">
+          <camera>
+            <horizontal_fov>3.14</horizontal_fov>
+            <image>
+              <width>1280</width>
+              <height>720</height>
+            </image>
+            <clip>
+              <near>0.1</near>
+              <far>100</far>
+            </clip>
+            <lens>
+              <type>custom</type>
+              <custom_function>
+                <c1>1.05</c1>
+                <c2>4</c2>
+                <f>1.0</f>
+                <fun>tan</fun>
+              </custom_function>
+              <scale_to_hfov>true</scale_to_hfov>
+              <cutoff_angle>3.1415</cutoff_angle>
+              <env_texture_size>1024</env_texture_size>
+            </lens>
+          </camera>
+          <always_on>1</always_on>
+          <update_rate>10</update_rate>
+          <visualize>1</visualize>
+          <topic>camera_right</topic>
+        </sensor>
+  </gazebo>
+  <joint name="camera_right_joint" type="fixed">
     <parent link="t265_link"/>
-    <child link="camera_left_optical_link"/>
-    <origin rpy="3.14 0 0" xyz="-0.0354 0 0"/>
-  </joint>
-  <gazebo reference="camera_left_link">
-      <sensor name="camera_left" type="camera">
-        <camera>
-          <horizontal_fov>1.75</horizontal_fov> <!-- ~100 degrees -->
-          <image>
-            <width>640</width> <!-- Increased resolution for better fidelity -->
-            <height>480</height>
-          </image>
-          <clip>
-            <near>0.1</near>
-            <far>100</far>
-          </clip>
-          <!-- Add camera_info_topic -->
-          <camera_info_topic>camera_left/camera_info</camera_info_topic>
-          <!-- Add frame_id -->
-          <optical_frame_id>camera_left_optical_link</optical_frame_id>
-        </camera>
-        <always_on>1</always_on>
-        <update_rate>30</update_rate>
-        <visualize>true</visualize>
-        <topic>camera_left</topic>
-      </sensor>
-  </gazebo>
-  <link name="camera_right_link">
-    <!-- <origin rpy="0 0 0" xyz="0.10 -0.03 0.05"/> -->
-    <inertial>
-      <mass value="0.1"/>
-      <inertia ixx="0.000166667" iyy="0.000166667" izz="0.000166667" ixy="0" ixz="0" iyz="0"/>
-    </inertial>
-    <visual>
-      <geometry>
-        <box size="0.02 0.02 0.02"/>
-      </geometry>
-      <gazebo>
-        <material>
-          <ambient>0 0 0 1</ambient>
-          <diffuse>0 0 0 1</diffuse>
-          <specular>0 0 0 1</specular>
-        </material>
-      </gazebo>
-    </visual>
-    <collision name="collision">
-      <geometry>
-        <box size="0.02 0.02 0.02"/>
-      </geometry>
-    </collision>
-  </link>
-  <joint name="camera_right_joint" type="fixed">
-    <parent link="camera_left_link"/>
     <child link="camera_right_link"/>
-    <origin rpy="0 1.57 0" xyz="0 0 0"/>
-  </joint>
-  <link name="camera_right_optical_link">
-    <!-- <origin rpy="0 0 0" xyz="0.10 -0.03 0.05"/> -->
-    <inertial>
-      <mass value="0.1"/>
-      <inertia ixx="0.000166667" iyy="0.000166667" izz="0.000166667" ixy="0" ixz="0" iyz="0"/>
-    </inertial>
-    <visual>
-      <geometry>
-        <box size="0.02 0.02 0.02"/>
-      </geometry>
-      <gazebo>
-        <material>
-          <ambient>0 0 0 1</ambient>
-          <diffuse>0 0 0 1</diffuse>
-          <specular>0 0 0 1</specular>
-        </material>
-      </gazebo>
-    </visual>
-    <collision name="collision">
-      <geometry>
-        <box size="0.02 0.02 0.02"/>
-      </geometry>
-    </collision>
-  </link>
-  <joint name="camera_right_optical_joint" type="fixed">
-    <parent link="t265_link"/>
-    <child link="camera_right_optical_link"/>
-    <origin rpy="3.14 0 0" xyz="0.0354 0 0"/>
-  </joint>
-  <gazebo reference="camera_right_link">
-      <sensor name="camera_right" type="camera">
-        <camera>
-          <horizontal_fov>1.75</horizontal_fov> <!-- ~100 degrees -->
-          <image>
-            <width>640</width> <!-- Increased resolution for better fidelity -->
-            <height>480</height>
-          </image>
-          <clip>
-            <near>0.1</near>
-            <far>100</far>
-          </clip>
-          <!-- Add camera_info_topic -->
-          <camera_info_topic>camera_right/camera_info</camera_info_topic>
-          <!-- Add frame_id -->
-          <optical_frame_id>camera_right_optical_link</optical_frame_id>
-        </camera>
-        <always_on>1</always_on>
-        <update_rate>30</update_rate>
-        <visualize>true</visualize>
-        <topic>camera_right</topic>
-      </sensor>
-  </gazebo>
+    <origin rpy="3.14 0 0" xyz="0.03 0 0"/>
+  </joint>
   <link name="t256_imu_link">
     <!-- <origin rpy="0 0 0" xyz="0 0 0"/> -->
@@ -412,9 +370,9 @@
     <sensor name="t265_imu_sensor" type="imu">
       <always_on>1</always_on>
-      <update_rate>200</update_rate>
+      <update_rate>100</update_rate>
       <visualize>true</visualize>
-      <topic>t265_imu</topic>
+      <topic>imu</topic>
       <enable_metrics>true</enable_metrics>
-      <gz_frame_id>t256_imu_link</gz_frame_id>
+      <gz_frame_id>imu_link</gz_frame_id>
     </sensor>
   </gazebo>
@@ -422,5 +380,5 @@
     <parent link="t265_link"/>
     <child link="t256_imu_link"/>
-    <origin rpy="3.14 0 3.14" xyz="-0.02 0 0"/>
+    <origin rpy="0 0 3.14" xyz="-0.02 0 0"/>
   </joint>
   <link name="lidar_link">
@@ -464,5 +422,5 @@
             <range>
               <min>0.08</min>
-              <max>100.0</max>
+              <max>12.0</max>
               <resolution>0.01</resolution>
             </range>
